File: amp/amp.kicad_pcb (KiCad board)
At the start: 2 copper layers, 387.4 x 193 mm, 48 parts, among them J1 Conn_01x03, J2 DUAL_RCA, SW1 SW_SPST, T1 Transformer_1P_1S, T2 Transformer_1P_1S, T3 Transformer_PT190.2, U1 6CY7, U2 6CY7, U3 6CA4

Commit message: save before branch
Parts:
- moved C7 179.9 mm to (222.2, 63.5)
- moved U2 4.58 mm to (259.1, 180.3)
- moved U3 2.54 mm to (363.2, 190.5)

Commit message: First draft layout done
Parts:
- J1: value Conn_01x03 -> Conn_01x05
- moved T3 144.9 mm to (276.9, 153.7), turned to 90 degrees
- moved L2 133.9 mm to (54.0, 52.1)
- moved L1 132.7 mm to (276.2, 50.8)
- moved R6 111.0 mm to (164.6, 193.5)
- moved R14 104.5 mm to (302.3, 196.8), turned to 180 degrees
- moved C6 95.6 mm to (287.0, 174.6)
- moved R10 83.8 mm to (203.8, 198.1)
- moved C4 83.2 mm to (216.5, 207.0)
- moved RV2 73.0 mm to (182.2, 215.9)
- moved T2 73.0 mm to (219.1, 114.9)
- moved U2 70.5 mm to (189.9, 193.7), turned to 0 degrees
- moved R7 63.5 mm to (189.9, 157.5)
- moved SW1 62.9 mm to (382.9, 205.7)
- moved C9 59.8 mm to (224.2, 152.4)
- moved F1 57.2 mm to (377.2, 67.3), turned to 180 degrees
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Connections:
- J1 pad 4: (no net) -> Earth_Protective
- J1 pad 5: (no net) -> Earth_Protective
- J2 pad 5: (no net) -> Earth
- J2 pad 6: (no net) -> Earth
- RV1 pad 1: Net-(J2-Pad1) -> Earth
- RV1 pad 3: Earth -> Net-(J2-Pad1)
- RV2 pad 1: Net-(J2-Pad3) -> Earth
- RV2 pad 3: Earth -> Net-(J2-Pad3)
- T1 pad 3: (no net) -> Net-(T1-Pad3)
- T2 pad 3: (no net) -> Net-(T2-Pad3)
- U1 pad 4: Net-(R13-Pad1) -> Net-(R12-Pad1)
- U1 pad 5: Net-(R12-Pad1) -> Net-(R13-Pad1)
- U3 pad 1: Net-(T3-Pad4) -> Net-(T3-Pad7)
- U3 pad 4: Net-(R14-Pad1) -> Net-(T3-Pad10)
- U3 pad 5: Net-(T3-Pad10) -> Net-(R14-Pad1)
- U3 pad 7: Net-(T3-Pad7) -> Net-(T3-Pad4)
Routing:
- net Earth: track 0.00 -> 693.1 mm
- net Net-(R13-Pad1): track 0.00 -> 284.4 mm
- net Net-(R12-Pad1): track 0.00 -> 276.0 mm, vias 0 -> 2
- net Net-(C7-Pad1): track 0.00 -> 239.0 mm
- net VBUS: track 0.00 -> 176.1 mm
- net HT: track 0.00 -> 163.7 mm
- net NEUT: track 0.00 -> 160.6 mm
- net Net-(F1-Pad1): track 0.00 -> 150.8 mm
- net LINE: track 0.00 -> 132.4 mm
- net Net-(T3-Pad10): track 0.00 -> 102.0 mm
- net Net-(R14-Pad1): track 0.00 -> 100.2 mm
- net Net-(LS1-Pad2): track 0.00 -> 90.7 mm
- net Net-(LS2-Pad2): track 0.00 -> 88.1 mm
- net Net-(T3-Pad4): track 0.00 -> 83.7 mm
- net Net-(T3-Pad7): track 0.00 -> 80.6 mm
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- added copper zone on B.Cu, net Earth
- added copper zone on B.Cu, net Earth_Protective

Commit message: Candidate for first build
Parts:
- SW1: value SW_SPST -> SW_SPST_GND
- moved J1 89.0 mm to (399.5, 127.3), turned to 90 degrees
- moved R11 68.2 mm to (370.6, 35.3), turned to 270 degrees
- moved C5 52.5 mm to (359.9, 45.2), turned to 90 degrees
- moved SW1 0.13 mm to (382.8, 205.7)
Connections:
- SW1 pad 4: (no net) -> Earth_Protective
- SW1 pad 5: (no net) -> Earth_Protective
Routing:
- net Net-(C6-Pad1): track 30.9 -> 154.3 mm
- net Earth: track 693.1 -> 749.2 mm
- net NEUT: track 160.6 -> 114.5 mm
- net /L: track 29.8 -> 74.3 mm
- net Net-(J2-Pad3): track 62.9 -> 69.3 mm
- net Net-(F1-Pad1): track 150.8 -> 149.1 mm
Other:
- board text added: "155H"
- board text added: "6CY7 Stereo Amplifier Circuit: Cascade Tubes PCB: E. Hazen 2021-01-02"
- board text added: "AC In 125V"
- board text added: "Fuse"
- board text added: "L"
- board text added: "L Spkr"
- board text added: "L Vol"
- board text added: "Line Input"
- board text added: "OT8SE"
- board text added: "PT190.2"
- board text added: "R"
- board text added: "R Spkr"
- board text added: "R Vol"

Commit message: Change to 6-32 mounting holes
Parts:
- H1, H2, H3, H4, H5, H6: footprint MountingHole:MountingHole_6.4mm_M6_Pad -> MountingHolesInch:Mtg6-32
- moved H3 23.5 mm to (261.6, 34.9)
- moved L1 15.2 mm to (291.5, 50.8)
- moved C5 12.1 mm to (372.0, 44.6)
- moved R11 12.1 mm to (382.7, 34.7)
Routing:
- net Earth_Protective: track 80.0 -> 50.5 mm
- net Net-(C7-Pad1): track 239.0 -> 254.5 mm
- net Net-(C6-Pad1): track 154.3 -> 160.6 mm
- net Earth: track 749.2 -> 755.0 mm
- net Net-(J2-Pad1): track 46.7 -> 45.1 mm
