File: amp/amp.sch (KiCad schematic (older format))
At the start: 42 parts, among them J1 Conn_01x03, J2 DUAL_RCA, SW1 SW_SPST, T1 Transformer_1P_1S, T2 Transformer_1P_1S, T3 Transformer_PT190.2, U1 6CY7, U2 6CY7, U3 6CA4

Commit message: First try at placement
Parts:
- removed C4: 100uF, Capacitor_THT:CP_Radial_D8.0mm_P3.50mm, symbol Device:C
- added C4: 100uF, Capacitor_THT:CP_Radial_D8.0mm_P3.50mm, symbol Device:CP
- added H1, H2, H3, H4, H5, H6: MTG, MountingHole:MountingHole_6.4mm_M6_Pad, symbol Mechanical:MountingHole_Pad
- C1: footprint (none) -> Capacitor_THT:C_Axial_L17.0mm_D6.5mm_P20.00mm_Horizontal; CatNo C-UD0033-630 -> 1572-1715-ND; Vendor AES -> DigiKey
- C3: footprint (none) -> Capacitor_THT:C_Axial_L17.0mm_D6.5mm_P20.00mm_Horizontal; CatNo (none) -> 1572-1715-ND; Vendor (none) -> DigiKey
- C5: value 10nF XYZ -> 5nF 400V Y4; footprint (none) -> Capacitor_THT:C_Disc_D11.0mm_W5.0mm_P10.00mm; CatNo (none) -> 125LD50-R-ND; Vendor (none) -> DigiKey
- C6: footprint Capacitor_THT:C_Radial_D12.5mm_H25.0mm_P5.00mm -> Capacitor_THT:CP_Radial_D12.5mm_P5.00mm
- C7, C8, C9: footprint (none) -> Capacitor_THT:CP_Radial_D18.0mm_P7.50mm
- J2: footprint (none) -> RCA_jack:PJRAS2X1S01AUX
- LS1, LS2: footprint (none) -> BindingPost:Keystone_4109; CatNo S-H263 -> 36-4109-ND; Vendor AES -> DigiKey
- R11: Vendor (none) -> DigiKey
- RV1, RV2: footprint (none) -> POT:P260P-D1BS3CA
- T1, T2: symbol Device:Transformer_1P_1S -> my_tubes:Transformer_1P_SS
Connections:
- net Earth: now also C4.2
- net VBUS: now also C9.1, L3.2
- net at T1.3 (IN_7K): no longer LS1.2
- net at R10.1, U2.9 (K): now also C4.1
- net at T2.3 (IN_7K): no longer LS2.2
- net at C6.1, U3.3 (K): now also L1.2; no longer L1.1
- net at C7.1, L2.1, L3.1: now also L1.1; no longer L1.2
- net E renamed Earth_Protective
- net Earth_Protective: now also H1.1, H2.1, H3.1, H4.1, H5.1, H6.1
- new net: LS1.2, T1.6 (OUT8)
- new net: LS2.2, T2.6 (OUT8)
Other:
- moved on the sheet: L1
Changed lines of the file:
@@
 F 0 "RV1" H 6357 2571 50  0000 R CNN
 F 1 "100k_audio" V 6350 2300 50  0000 R CNN
-F 2 "" H 6425 2525 50  0001 C CNN
+F 2 "POT:P260P-D1BS3CA" H 6425 2525 50  0001 C CNN
 F 3 "~" H 6425 2525 50  0001 C CNN
 F 4 "987-1330-ND" H 6400 3050 50  0000 C CNN "CatNo"
@@
 F 0 "C1" V 7258 2025 50  0000 C CNN
 F 1 ".0033uF" V 7349 2025 50  0000 C CNN
-F 2 "" H 7638 1875 50  0001 C CNN
+F 2 "Capacitor_THT:C_Axial_L17.0mm_D6.5mm_P20.00mm_Horizontal" H 7638 1875 50  0001 C CNN
 F 3 "~" H 7600 2025 50  0001 C CNN
-F 4 "C-UD0033-630" V 7440 2025 50  0000 C CNN "CatNo"
-F 5 "AES" V 7600 2025 50  0001 C CNN "Vendor"
+F 4 "1572-1715-ND" V 7440 2025 50  0000 C CNN "CatNo"
+F 5 "DigiKey" V 7600 2025 50  0001 C CNN "Vendor"
 	1    7600 2025
 	0    1    1    0
@@
 	9575 3325 9575 2875
 $Comp
-L Device:Transformer_1P_1S T1
+L my_tubes:Transformer_1P_SS T1
 U 1 1 5FEFBAC8
 P 9900 1425
@@
 F 0 "LS1" H 10820 1391 50  0000 L CNN
 F 1 "Speaker" H 10820 1300 50  0000 L CNN
-F 2 "" H 10650 1150 50  0001 C CNN
+F 2 "BindingPost:Keystone_4109" H 10650 1150 50  0001 C CNN
 F 3 "~" H 10640 1300 50  0001 C CNN
-F 4 "S-H263" H 10820 1209 50  0000 L CNN "CatNo"
-F 5 "AES" H 10650 1350 50  0001 C CNN "Vendor"
+F 4 "36-4109-ND" H 10820 1209 50  0000 L CNN "CatNo"
+F 5 "DigiKey" H 10650 1350 50  0001 C CNN "Vendor"
 	1    10650 1350
 	1    0    0    -1
@@
 Wire Wire Line
 	9250 1425 9500 1425
-Wire Wire Line
-	9500 1425 9500 1625
 $Comp
 L my_tubes:6CY7 U2
@@
 F 0 "RV2" H 6332 5271 50  0000 R CNN
 F 1 "100k_audio" V 6250 5200 50  0000 R CNN
-F 2 "" H 6400 5225 50  0001 C CNN
+F 2 "POT:P260P-D1BS3CA" H 6400 5225 50  0001 C CNN
 F 3 "~" H 6400 5225 50  0001 C CNN
 F 4 "987-1330-ND" H 5800 5175 50  0000 C CNN "CatNo"
@@
 F 0 "C3" V 7323 4725 50  0000 C CNN
 F 1 ".0033uF" V 7414 4725 50  0000 C CNN
-F 2 "" H 7613 4575 50  0001 C CNN
+F 2 "Capacitor_THT:C_Axial_L17.0mm_D6.5mm_P20.00mm_Horizontal" H 7613 4575 50  0001 C CNN
 F 3 "~" H 7575 4725 50  0001 C CNN
+F 4 "1572-1715-ND" V 7225 4800 50  0000 C CNN "CatNo"
+F 5 "DigiKey" V 7575 4725 50  0001 C CNN "Vendor"
 	1    7575 4725
 	0    1    1    0
@@
 F 2 "Resistor_THT:R_Axial_DIN0414_L11.9mm_D4.5mm_P15.24mm_Horizontal" V 8565 4715 50  0001 C CNN
 F 3 "~" H 8525 4725 50  0001 C CNN
-F 4 "BC4520CT-ND" H 8525 4725 50  0001 C CNN "CatNo"
+F 4 "BC4520CT-ND" V 8175 4725 50  0000 C CNN "CatNo"
 	1    8525 4725
 	0    1    1    0
@@
 Wire Wire Line
 	6950 6050 6950 5975
-$Comp
-L Device:C C4
-U 1 1 5FF17473
-P 9550 5425
-F 0 "C4" H 9435 5334 50  0000 R CNN
-F 1 "100uF" H 9435 5425 50  0000 R CNN
-F 2 "Capacitor_THT:CP_Radial_D8.0mm_P3.50mm" H 9588 5275 50  0001 C CNN
-F 3 "~" H 9550 5425 50  0001 C CNN
-F 4 "732-8666-1-ND" H 9435 5516 50  0000 R CNN "CatNo"
-F 5 "DigiKey" H 9550 5425 50  0001 C CNN "Vendor"
-	1    9550 5425
-	-1   0    0    1
-$EndComp
 Wire Wire Line
 	9550 5275 9550 5225
@@
 	9550 6025 9550 5575
 $Comp
-L Device:Transformer_1P_1S T2
+L my_tubes:Transformer_1P_SS T2
 U 1 1 5FF1748C
 P 9875 4125
@@
 F 0 "LS2" H 10820 4091 50  0000 L CNN
 F 1 "Speaker" H 10820 4000 50  0000 L CNN
-F 2 "" H 10650 3850 50  0001 C CNN
+F 2 "BindingPost:Keystone_4109" H 10650 3850 50  0001 C CNN
 F 3 "~" H 10640 4000 50  0001 C CNN
-F 4 "S-H263" H 10820 3909 50  0000 L CNN "CatNo"
-F 5 "AES" H 10650 4050 50  0001 C CNN "Vendor"
+F 4 "36-4109-ND" H 10820 3909 50  0000 L CNN "CatNo"
+F 5 "DigiKey" H 10650 4050 50  0001 C CNN "Vendor"
 	1    10650 4050
 	1    0    0    -1
@@
 Wire Wire Line
 	9225 4125 9475 4125
-Wire Wire Line
-	9475 4125 9475 4325
 $Comp
 L my_tubes:6CY7 U2
@@
 U 1 1 5FFB3E15
 P 3950 2850
-F 0 "L1" V 4231 2850 50  0000 C CNN
-F 1 "5H/156L" V 4140 2850 50  0000 C CNN
+F 0 "L1" V 3775 2825 50  0000 C CNN
+F 1 "5H/156L" V 3875 2850 50  0000 C CNN
 F 2 "Hammond-L:156L" H 3950 2850 50  0001 C CNN
 F 3 "~" H 3950 2850 50  0001 C CNN
-F 4 "HM3516-ND" V 4049 2850 50  0000 C CNN "CatNo"
+F 4 "HM3516-ND" V 4625 2875 50  0000 C CNN "CatNo"
 F 5 "DigiKey" V 3950 2850 50  0001 C CNN "Vendor"
 	1    3950 2850
-	0    -1   -1   0
+	0    1    1    0
 $EndComp
 Wire Wire Line
@@
 	1    0    0    -1
 $EndComp
-Wire Wire Line
-	4775 3425 5175 3425
 Wire Wire Line
 	5175 3425 5175 3375
@@
 P 1350 2250
 F 0 "C5" H 1250 2450 50  0000 R CNN
-F 1 "10nF XYZ" H 1275 2350 50  0000 R CNN
-F 2 "" H 1388 2100 50  0001 C CNN
+F 1 "5nF 400V Y4" H 1275 2350 50  0000 R CNN
+F 2 "Capacitor_THT:C_Disc_D11.0mm_W5.0mm_P10.00mm" H 1388 2100 50  0001 C CNN
 F 3 "~" H 1350 2250 50  0001 C CNN
+F 4 "125LD50-R-ND" H 775 2450 50  0000 C CNN "CatNo"
+F 5 "DigiKey" H 1350 2250 50  0001 C CNN "Vendor"
 	1    1350 2250
 	-1   0    0    1
@@
 F 2 "Resistor_THT:R_Axial_DIN0414_L11.9mm_D4.5mm_P15.24mm_Horizontal" V 1015 2240 50  0001 C CNN
 F 3 "~" H 975 2250 50  0001 C CNN
-F 4 "BC4517CT-ND" H 975 2250 50  0001 C CNN "CatNo"
+F 4 "BC4517CT-ND" H 975 1950 50  0000 C CNN "CatNo"
+F 5 "DigiKey" H 975 2250 50  0001 C CNN "Vendor"
 	1    975  2250
 	1    0    0    -1
@@
 F 0 "J2" H 6188 4280 50  0000 C CNN
 F 1 "DUAL_RCA" H 6300 4200 50  0000 C CNN
-F 2 "" H 5975 3925 50  0001 C CNN
+F 2 "RCA_jack:PJRAS2X1S01AUX" H 5975 3925 50  0001 C CNN
 F 3 "" H 5975 3925 50  0001 C CNN
 F 4 "SC1858-ND" H 6275 4100 50  0000 C CNN "CatNo"
@@
 F 0 "C6" H 3843 3191 50  0000 L CNN
 F 1 "33uF" H 3843 3100 50  0000 L CNN
-F 2 "Capacitor_THT:C_Radial_D12.5mm_H25.0mm_P5.00mm" H 3763 2950 50  0001 C CNN
+F 2 "Capacitor_THT:CP_Radial_D12.5mm_P5.00mm" H 3763 2950 50  0001 C CNN
 F 3 "~" H 3725 3100 50  0001 C CNN
 F 4 "493-12996-1-ND" V 3725 3500 50  0000 L CNN "CatNo"
@@
 F 0 "C7" H 4293 3146 50  0000 L CNN
 F 1 "100uF 350V" V 4250 3650 50  0000 L CNN
-F 2 "" H 4213 2950 50  0001 C CNN
+F 2 "Capacitor_THT:CP_Radial_D18.0mm_P7.50mm" H 4213 2950 50  0001 C CNN
 F 3 "~" H 4175 3100 50  0001 C CNN
 F 4 "1189-4068-ND" V 4175 3775 50  0000 C CNN "CatNo"
@@
 F 0 "C8" H 4868 3146 50  0000 L CNN
 F 1 "100uF 350V" V 4825 3650 50  0000 L CNN
-F 2 "" H 4788 2950 50  0001 C CNN
+F 2 "Capacitor_THT:CP_Radial_D18.0mm_P7.50mm" H 4788 2950 50  0001 C CNN
 F 3 "~" H 4750 3100 50  0001 C CNN
 F 4 "1189-4068-ND" V 4750 3775 50  0000 C CNN "CatNo"
@@
 F 0 "C9" H 4975 3700 50  0000 L CNN
 F 1 "100uF 350V" V 4900 3350 50  0000 L CNN
-F 2 "" H 4788 3525 50  0001 C CNN
+F 2 "Capacitor_THT:CP_Radial_D18.0mm_P7.50mm" H 4788 3525 50  0001 C CNN
 F 3 "~" H 4750 3675 50  0001 C CNN
 F 4 "1189-4068-ND" V 4575 3525 50  0000 C CNN "CatNo"
@@
 Wire Wire Line
 	1875 2175 3225 2175
+Wire Wire Line
+	4750 3425 5175 3425
+Connection ~ 4750 3425
+$Comp
+L Device:CP C4
+U 1 1 5FF97797
+P 9550 5425
+F 0 "C4" V 9668 5471 50  0000 L CNN
+F 1 "100uF" H 9675 5375 50  0000 L CNN
+F 2 "Capacitor_THT:CP_Radial_D8.0mm_P3.50mm" H 9588 5275 50  0001 C CNN
+F 3 "~" H 9550 5425 50  0001 C CNN
+F 4 "732-8666-1-ND" H 10000 5275 50  0000 C CNN "CatNo"
+F 5 "DigiKey" H 9550 5425 50  0001 C CNN "Vendor"
+	1    9550 5425
+	1    0    0    -1
+$EndComp
+$Comp
+L Mechanical:MountingHole_Pad H1
+U 1 1 6001190D
+P 1175 7075
+F 0 "H1" H 1275 7124 50  0000 L CNN
+F 1 "MTG" H 1275 7050 50  0000 L CNN
+F 2 "MountingHole:MountingHole_6.4mm_M6_Pad" H 1175 7075 50  0001 C CNN
+F 3 "~" H 1175 7075 50  0001 C CNN
+	1    1175 7075
+	1    0    0    -1
+$EndComp
+$Comp
+L Mechanical:MountingHole_Pad H2
+U 1 1 6001261A
+P 1550 7075
+F 0 "H2" H 1650 7124 50  0000 L CNN
+F 1 "MTG" H 1650 7050 50  0000 L CNN
+F 2 "MountingHole:MountingHole_6.4mm_M6_Pad" H 1550 7075 50  0001 C CNN
+F 3 "~" H 1550 7075 50  0001 C CNN
+	1    1550 7075
+	1    0    0    -1
+$EndComp
+$Comp
+L Mechanical:MountingHole_Pad H3
+U 1 1 60018F38
+P 1950 7075
+F 0 "H3" H 2050 7124 50  0000 L CNN
+F 1 "MTG" H 2050 7050 50  0000 L CNN
+F 2 "MountingHole:MountingHole_6.4mm_M6_Pad" H 1950 7075 50  0001 C CNN
+F 3 "~" H 1950 7075 50  0001 C CNN
+	1    1950 7075
+	1    0    0    -1
+$EndComp
+$Comp
+L Mechanical:MountingHole_Pad H4
+U 1 1 60019788
+P 2325 7075
+F 0 "H4" H 2425 7124 50  0000 L CNN
+F 1 "MTG" H 2425 7050 50  0000 L CNN
+F 2 "MountingHole:MountingHole_6.4mm_M6_Pad" H 2325 7075 50  0001 C CNN
+F 3 "~" H 2325 7075 50  0001 C CNN
+	1    2325 7075
+	1    0    0    -1
+$EndComp
+$Comp
+L Mechanical:MountingHole_Pad H5
+U 1 1 600204DC
+P 2700 7075
+F 0 "H5" H 2800 7124 50  0000 L CNN
+F 1 "MTG" H 2800 7050 50  0000 L CNN
+F 2 "MountingHole:MountingHole_6.4mm_M6_Pad" H 2700 7075 50  0001 C CNN
+F 3 "~" H 2700 7075 50  0001 C CNN
+	1    2700 7075
+	1    0    0    -1
+$EndComp
+$Comp
+L Mechanical:MountingHole_Pad H6
+U 1 1 600204E2
+P 3075 7075
+F 0 "H6" H 3175 7124 50  0000 L CNN
+F 1 "MTG" H 3175 7050 50  0000 L CNN
+F 2 "MountingHole:MountingHole_6.4mm_M6_Pad" H 3075 7075 50  0001 C CNN
+F 3 "~" H 3075 7075 50  0001 C CNN
+	1    3075 7075
+	1    0    0    -1
+$EndComp
+Wire Wire Line
+	1175 7175 1175 7300
+Wire Wire Line
+	1175 7300 1550 7300
+Wire Wire Line
+	1550 7300 1550 7175
+Wire Wire Line
+	1550 7300 1950 7300
+Wire Wire Line
+	1950 7300 1950 7175
+Connection ~ 1550 7300
+Wire Wire Line
+	1950 7300 2325 7300
+Wire Wire Line
+	2325 7300 2325 7175
+Connection ~ 1950 7300
+Wire Wire Line
+	2325 7300 2700 7300
+Wire Wire Line
+	2700 7300 2700 7175
+Connection ~ 2325 7300
+Wire Wire Line
+	2700 7300 3075 7300
+Wire Wire Line
+	3075 7300 3075 7175
+Connection ~ 2700 7300
+$Comp
+L power:Earth_Protective #PWR0101
+U 1 1 60049BC3
+P 700 1975
+F 0 "#PWR0101" H 950 1725 50  0001 C CNN
+F 1 "Earth_Protective" H 1150 1825 50  0001 C CNN
+F 2 "" H 700 1875 50  0001 C CNN
+F 3 "~" H 700 1875 50  0001 C CNN
+	1    700  1975
+	1    0    0    -1
+$EndComp
+Wire Wire Line
+	700  1975 975  1975
+Connection ~ 975  1975
+$Comp
+L power:Earth_Protective #PWR0102
+U 1 1 60051CEC
+P 1175 7300
+F 0 "#PWR0102" H 1425 7050 50  0001 C CNN
+F 1 "Earth_Protective" H 1625 7150 50  0001 C CNN
+F 2 "" H 1175 7200 50  0001 C CNN
+F 3 "~" H 1175 7200 50  0001 C CNN
+	1    1175 7300
+	1    0    0    -1
+$EndComp
+Connection ~ 1175 7300
 $EndSCHEMATC
